File: RFM26W Breakout Board/rfm26w_breakout_board.brd (EAGLE design)
At the start: 24.1 x 30.5 mm, 5 parts, among them X1 BU-SMA

Commit message: Added Gerber files.
Parts:
- added U$3: (no value), KaiBader-Logos:OSHW-LOGO-S
Changed lines of the file:
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@@
 <layer number="97" name="Info" color="7" fill="1" visible="no" active="no"/>
 <layer number="98" name="Guide" color="6" fill="1" visible="no" active="no"/>
+<layer number="99" name="SpiceOrder" color="7" fill="1" visible="no" active="no"/>
 <layer number="100" name="Muster" color="7" fill="1" visible="no" active="no"/>
 <layer number="101" name="Patch_Top" color="12" fill="4" visible="no" active="yes"/>
@@
 </class>
 </classes>
-<designrules name="ITEADstudio_DRC">
-<description language="de">&lt;b&gt;EAGLE Design Rules&lt;/b&gt;
-&lt;p&gt;
-Die Standard-Design-Rules sind so gewählt, dass sie für
-die meisten Anwendungen passen. Sollte ihre Platine
-besondere Anforderungen haben, treffen Sie die erforderlichen
-Einstellungen hier und speichern die Design Rules unter
-einem neuen Namen ab.</description>
-<description language="en">&lt;b&gt;EAGLE Design Rules&lt;/b&gt;
-&lt;p&gt;
-The default Design Rules have been set to cover
-a wide range of applications. Your particular design
-may have different requirements, so please make the
-necessary adjustments and save your customized
-design rules under a new name.</description>
-<description language="zh">&lt;b&gt;Seeed Studio EAGLE Design Rules&lt;/b&gt;
-</description>
+<designrules name="dirt_cheap_dirty_boards.v1">
+<description language="en">&lt;b&gt;Dirty Cheap Dirty Board Design Rules&lt;/b&gt;
+&lt;br&gt;
+&lt;br&gt;Min width/Spacing: 5/5mil
+&lt;br&gt;Min diameter of finished hole 12mil</description>
 <param name="layerSetup" value="(1*16)"/>
-<param name="mtCopper" value="0.035mm 0.035mm 0.035mm 0.035mm 0.035mm 0.035mm 0.035mm 0.035mm 0.035mm 0.035mm 0.035mm 0.035mm 0.035mm 0.035mm 0.035mm 0.035mm"/>
-<param name="mtIsolate" value="1.5mm 0.15mm 0.2mm 0.15mm 0.2mm 0.15mm 0.2mm 0.15mm 0.2mm 0.15mm 0.2mm 0.15mm 0.2mm 0.15mm 0.2mm"/>
-<param name="mdWireWire" value="6mil"/>
-<param name="mdWirePad" value="6mil"/>
-<param name="mdWireVia" value="6mil"/>
-<param name="mdPadPad" value="6mil"/>
-<param name="mdPadVia" value="6mil"/>
-<param name="mdViaVia" value="6mil"/>
+<param name="mtCopper" value="0.035mm 0.0175mm 0.035mm 0.035mm 0.035mm 0.035mm 0.035mm 0.035mm 0.035mm 0.035mm 0.035mm 0.035mm 0.035mm 0.035mm 0.0175mm 0.035mm"/>
+<param name="mtIsolate" value="1.5mm 1.1mm 0.2mm 0.15mm 0.2mm 0.15mm 0.2mm 0.15mm 0.2mm 0.15mm 0.2mm 0.15mm 0.2mm 0.15mm 0.2mm"/>
+<param name="mdWireWire" value="5mil"/>
+<param name="mdWirePad" value="5mil"/>
+<param name="mdWireVia" value="5mil"/>
+<param name="mdPadPad" value="5mil"/>
+<param name="mdPadVia" value="5mil"/>
+<param name="mdViaVia" value="5mil"/>
 <param name="mdSmdPad" value="0mil"/>
 <param name="mdSmdVia" value="0mil"/>
@@
 <param name="mdDrill" value="10mil"/>
 <param name="mdSmdStop" value="0mil"/>
-<param name="msWidth" value="6mil"/>
+<param name="msWidth" value="5mil"/>
 <param name="msDrill" value="12mil"/>
 <param name="msMicroVia" value="12mil"/>
@@
 <param name="mlMinCreamFrame" value="0mil"/>
 <param name="mlMaxCreamFrame" value="0mil"/>
-<param name="mlViaStopLimit" value="100mil"/>
+<param name="mlViaStopLimit" value="25mil"/>
 <param name="srRoundness" value="0"/>
 <param name="srMinRoundness" value="0mil"/>
@@
 <attribute name="VALUE" x="19.05" y="20.955" size="1.27" layer="27" rot="R270"/>
 </element>
+<element name="U$3" library="KaiBader-Logos" package="OSHW-LOGO-S" value="" x="18.034" y="24.257"/>
 </elements>
 <signals>
@@
 <contactref element="JP2" pad="4"/>
 <wire x1="11.065" y1="18.795" x2="11.065" y2="20.05" width="0.3048" layer="1"/>
-<wire x1="11.065" y1="20.05" x2="9.525" y2="21.59" width="0.508" layer="1"/>
-<wire x1="9.525" y1="21.59" x2="6.62" y2="21.59" width="0.508" layer="1"/>
-<wire x1="6.62" y1="21.59" x2="5.715" y2="22.495" width="0.508" layer="1"/>
+<wire x1="11.065" y1="20.05" x2="9.525" y2="21.59" width="0.6096" layer="1"/>
+<wire x1="9.525" y1="21.59" x2="6.62" y2="21.59" width="0.6096" layer="1"/>
+<wire x1="6.62" y1="21.59" x2="5.715" y2="22.495" width="0.6096" layer="1"/>
 <wire x1="11.065" y1="18.795" x2="10.795" y2="18.795" width="0.3048" layer="1"/>
-<wire x1="10.795" y1="18.795" x2="10.795" y2="13.335" width="0.508" layer="1"/>
+<wire x1="10.795" y1="18.795" x2="10.795" y2="13.335" width="0.6096" layer="1"/>
 <via x="10.795" y="13.335" extent="1-16" drill="0.6"/>
-<wire x1="10.795" y1="13.335" x2="19.685" y2="13.335" width="0.508" layer="16"/>
-<wire x1="19.685" y1="13.335" x2="20.955" y2="12.065" width="0.508" layer="16"/>
-<wire x1="20.955" y1="12.065" x2="22.225" y2="12.065" width="0.508" layer="16"/>
+<wire x1="10.795" y1="13.335" x2="19.685" y2="13.335" width="0.6096" layer="16"/>
+<wire x1="19.685" y1="13.335" x2="20.955" y2="12.065" width="0.6096" layer="16"/>
+<wire x1="20.955" y1="12.065" x2="22.225" y2="12.065" width="0.6096" layer="16"/>
 </signal>
 <signal name="TX-ANT">
@@
 <contactref element="PCB" pad="ANT"/>
 <contactref element="X1" pad="1"/>
-<wire x1="19.065" y1="18.795" x2="19.065" y2="22.21" width="0.508" layer="1"/>
-<wire x1="19.065" y1="22.21" x2="15.24" y2="26.035" width="0.508" layer="1"/>
-<wire x1="15.24" y1="26.035" x2="12.065" y2="26.035" width="0.508" layer="1"/>
+<wire x1="19.065" y1="18.795" x2="19.065" y2="22.21" width="0.6096" layer="1"/>
+<wire x1="19.065" y1="22.21" x2="15.24" y2="26.035" width="0.6096" layer="1"/>
+<wire x1="15.24" y1="26.035" x2="12.065" y2="26.035" width="0.6096" layer="1"/>
 </signal>
 </signals>
